File: Hardware/PCB/main_board/main_board.kicad_pcb (KiCad board)
At the start: 2 copper layers, 61 parts, among them J1 SWD, J2 USB_A, J3 DIN-5_180degree, J4 USB_B, Q1 BC547, SW1 SW_Push, SW10 SW_Push, SW11 SW_Push, SW2 SW_Push, SW3 SW_Push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

Commit message: Place HMI
Parts:
- removed RV1, RV10, RV11, RV12, RV13, RV14, RV2, RV3, RV4, RV5, RV6, RV7, RV8, RV9: 10k, Potentiometer_THT:Potentiometer_Alps_RK09K_Single_Vertical
- removed SW1, SW10, SW11, SW2, SW3, SW4, SW5, SW6, SW7, SW8, SW9: SW_Push, Button_Switch_THT:SW_PUSH_6mm_H13mm
- added BAR1: HDSP-4840_2, Display:HDSP-4840, F.Cu at (60.0, 57.5)
- added RV_ADSR_A1: 10k, Potentiometer_THT:Potentiometer_Alps_RK09K_Single_Vertical, F.Cu at (130.0, 100.0)
- added RV_ADSR_D1: 10k, Potentiometer_THT:Potentiometer_Alps_RK09K_Single_Vertical, F.Cu at (150.0, 100.0)
- added RV_ADSR_R1: 10k, Potentiometer_THT:Potentiometer_Alps_RK09K_Single_Vertical, F.Cu at (150.0, 120.0)
- added RV_ADSR_S1: 10k, Potentiometer_THT:Potentiometer_Alps_RK09K_Single_Vertical, F.Cu at (130.0, 120.0)
- added RV_DIST_DRIVE1: 10k, Potentiometer_THT:Potentiometer_Alps_RK09K_Single_Vertical, F.Cu at (110.0, 140.0)
- added RV_DIST_MIX1: 10k, Potentiometer_THT:Potentiometer_Alps_RK09K_Single_Vertical, F.Cu at (130.0, 140.0)
- added RV_DIST_TONE1: 10k, Potentiometer_THT:Potentiometer_Alps_RK09K_Single_Vertical, F.Cu at (150.0, 140.0)
- added RV_HPF_CUT1: 10k, Potentiometer_THT:Potentiometer_Alps_RK09K_Single_Vertical, F.Cu at (60.0, 160.0)
- added RV_HPF_RES1: 10k, Potentiometer_THT:Potentiometer_Alps_RK09K_Single_Vertical, F.Cu at (80.0, 160.0)
- added RV_LFO_DEPTH1: 10k, Potentiometer_THT:Potentiometer_Alps_RK09K_Single_Vertical, F.Cu at (60.0, 140.0)
- added RV_LFO_RATE1: 10k, Potentiometer_THT:Potentiometer_Alps_RK09K_Single_Vertical, F.Cu at (80.0, 140.0)
- added RV_OSC1_AMP1: 10k, Potentiometer_THT:Potentiometer_Alps_RK09K_Single_Vertical, F.Cu at (60.0, 100.0)
- added RV_OSC1_DET1: 10k, Potentiometer_THT:Potentiometer_Alps_RK09K_Single_Vertical, F.Cu at (60.0, 120.0)
- added RV_OSC2_AMP1: 10k, Potentiometer_THT:Potentiometer_Alps_RK09K_Single_Vertical, F.Cu at (80.0, 100.0)
- added RV_OSC2_DET1: 10k, Potentiometer_THT:Potentiometer_Alps_RK09K_Single_Vertical, F.Cu at (80.0, 120.0)
- added RV_OSC3_AMP1: 10k, Potentiometer_THT:Potentiometer_Alps_RK09K_Single_Vertical, F.Cu at (100.0, 100.0)
- added RV_OSC3_DET1: 10k, Potentiometer_THT:Potentiometer_Alps_RK09K_Single_Vertical, F.Cu at (100.0, 120.0)
- added RV_VOL1: R_POT_Dual, Potentiometer_THT:Potentiometer_Alps_RK09L_Double_Vertical, F.Cu at (150.0, 45.0)
- added SW_CTRL_DOWN1: SW_Push, Button_Switch_THT:SW_PUSH_6mm_H13mm, F.Cu at (130.0, 75.0)
- added SW_CTRL_LEFT1: SW_Push, Button_Switch_THT:SW_PUSH_6mm_H13mm, F.Cu at (120.0, 65.0)
- added SW_CTRL_OK1: SW_Push, Button_Switch_THT:SW_PUSH_6mm_H13mm, F.Cu at (130.0, 65.0)
- added SW_CTRL_RIGHT1: SW_Push, Button_Switch_THT:SW_PUSH_6mm_H13mm, F.Cu at (140.0, 65.0)
- added SW_CTRL_UP1: SW_Push, Button_Switch_THT:SW_PUSH_6mm_H13mm, F.Cu at (130.0, 55.0)
- added SW_OSC1_ON1: SW_Push, Button_Switch_THT:SW_PUSH_6mm_H13mm, F.Cu at (54.0, 65.0)
- added SW_OSC1_WAVE1: SW_Push, Button_Switch_THT:SW_PUSH_6mm_H13mm, F.Cu at (54.0, 75.0)
- added SW_OSC2_ON1: SW_Push, Button_Switch_THT:SW_PUSH_6mm_H13mm, F.Cu at (74.0, 65.0)
- added SW_OSC2_WAVE1: SW_Push, Button_Switch_THT:SW_PUSH_6mm_H13mm, F.Cu at (74.0, 75.0)
- added SW_OSC3_ON1: SW_Push, Button_Switch_THT:SW_PUSH_6mm_H13mm, F.Cu at (94.0, 65.0)
- added SW_OSC3_WAVE1: SW_Push, Button_Switch_THT:SW_PUSH_6mm_H13mm, F.Cu at (94.0, 75.0)
- moved J1 640.6 mm to (-110.0, 170.0)
- moved U2 638.6 mm to (-57.5, 147.5)
- moved Brd2 577.2 mm to (110.0, 45.0)
- moved Brd1 574.8 mm to (78.6, 45.0)
- moved C10 516.1 mm to (-32.6, 44.7)
- moved C12 516.1 mm to (-24.0, 44.8)
- moved C5 516.1 mm to (-80.9, 72.9)
- moved C6 516.1 mm to (-94.9, 38.5)
- moved C7 516.1 mm to (-62.5, 43.9)
- moved C8 516.1 mm to (-29.6, 41.2)
- moved C9 516.1 mm to (-34.9, 40.4)
- moved D1 516.1 mm to (-52.0, 47.3)
- moved FB1 516.1 mm to (-29.6, 39.2)
- moved FB2 516.1 mm to (-28.5, 46.3)
- moved J2 516.1 mm to (-91.3, 34.3)
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Routing:
- net Net-(C4-Pad2): track 57.0 -> 20.5 mm
- net Net-(C3-Pad1): track 31.9 -> 0.00 mm
- net +5VA: track 30.3 -> 18.9 mm
- net Net-(R2-Pad2): track 13.6 -> 3.63 mm
Other:
- board text added: "Indication d'echelle"
- board text removed: "Cuttof"
- board text removed: "Res"

Commit message: Place connectors
Parts:
- removed RV_DIST_MIX1: 10k, Potentiometer_THT:Potentiometer_Alps_RK09K_Single_Vertical
- moved J1 275.0 mm to (165.0, 166.3)
- moved U2 182.5 mm to (125.0, 147.5), turned to 180 degrees
- moved C6 160.1 mm to (65.1, 33.5)
- moved J2 160.1 mm to (68.7, 29.3)
- moved C7 145.1 mm to (82.5, 38.9)
- moved D1 145.1 mm to (93.0, 42.3)
- moved J3 145.1 mm to (89.2, 25.5)
- moved R8 145.1 mm to (93.0, 38.0)
- moved R9 145.1 mm to (85.9, 43.1)
- moved U3 145.1 mm to (87.5, 39.0)
- moved C14 144.8 mm to (122.5, 55.0)
- moved R6 115.8 mm to (-15.9, 178.0)
- moved R7 115.8 mm to (-19.7, 178.0)
- moved C1 115.8 mm to (-26.3, 169.1)
- moved C2 115.8 mm to (-19.7, 180.5)
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Other:
- board outline added: 150 x 177.5 mm
- board text removed: "Indication d'echelle"
