File: Hardware/PCB/main_board/main_board.kicad_pcb (KiCad board)
At the start: 4 copper layers, 140 x 125 mm, 157 parts, among them J1 SWD, J10 I2C_SDA, J11 UART_RX_MIDI, J12 Post_AB_amp, J13 Audio_out_jack, J14 +5V, J15 Post_VCF, J16 Post_buffer, J17 Post_FX, J19 Audio_MCU, J2 USB_A, J20 LFO_MCU, J21 GND, J22 GND, J23 +3.3V, J24 +5VA, J3 DIN-5_180degree, J4 USB_B, J5 I2C_SCL, J6 AudioJack3, J7 GND, J8 GND, J9 Pre_AB_amp, Q1 BC857B, Q2 BC847B, Q3 BC847B, Q4 BC857B, Q5 BC847B, U1 MCP6002-xSN, U2 LD1117S33TR_SOT223, U3 6N137, U4 RC4558, U5 MCP6002-xSN, U6 STM32F446RETx, Y1 Crystal

Commit message: Finish PCB routing
Parts:
- J1: footprint Connector_PinHeader_2.54mm:PinHeader_1x06_P2.54mm_Vertical -> Connector_PinHeader_2.54mm:PinHeader_1x05_P2.54mm_Vertical
- moved J1 95.0 mm to (88.6, 75.0), turned to 0 degrees
- moved C11 91.7 mm to (175.8, 52.0)
- moved C12 91.2 mm to (181.4, 51.0)
- moved FB2 90.5 mm to (175.8, 49.9), turned to 180 degrees
- moved C47 86.9 mm to (101.3, 64.5), turned to 180 degrees
- moved J24 83.1 mm to (165.9, 40.4)
- moved R34 78.0 mm to (99.4, 72.1), turned to 180 degrees
- moved C44 73.3 mm to (115.3, 63.7), turned to 90 degrees
- moved C46 72.5 mm to (99.4, 74.4), turned to 180 degrees
- moved C41 69.0 mm to (117.3, 63.7), turned to 270 degrees
- moved U6 68.0 mm to (108.5, 70.3), turned to 90 degrees
- moved C42 64.2 mm to (100.2, 82.9), turned to 270 degrees
- moved Y1 56.9 mm to (104.3, 82.0), turned to 0 degrees
- moved C43 49.3 mm to (104.6, 85.3)
- moved C48 49.1 mm to (114.8, 77.3), turned to 270 degrees
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Connections:
- J1 pad 1: /MCU/VDD_TARGET -> +3V3
Routing:
- net +3V3: track 15.2 -> 430.0 mm, vias 0 -> 10
- net +5VA: track 24.5 -> 211.6 mm, vias 0 -> 12
- net +5V: track 35.4 -> 193.3 mm
- net /MCU/ADC1_IN15: track 0.00 -> 135.0 mm, vias 0 -> 4
- net /MCU/ADC1_IN12: track 0.00 -> 127.1 mm, vias 0 -> 3
- net /MCU/ADC1_IN14: track 0.00 -> 106.8 mm
- net /MCU/ADC1_IN13: track 0.00 -> 104.8 mm, vias 0 -> 3
- net /MCU/ADC1_IN6: track 0.00 -> 100.8 mm, vias 0 -> 4
- net /MCU/ADC1_IN7: track 0.00 -> 88.7 mm, vias 0 -> 2
- net /MCU/ADC1_IN9: track 0.00 -> 87.8 mm
- net /MCU/ADC1_IN10: track 0.00 -> 87.4 mm, vias 0 -> 2
- net Net-(R18-Pad1): track 2.90 -> 86.2 mm
- net Net-(C18-Pad1): track 16.3 -> 99.5 mm, vias 0 -> 2
- net /MCU/ADC1_IN2: track 0.00 -> 77.0 mm
- net Net-(C3-Pad1): track 0.00 -> 74.9 mm
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- added copper zone on F.Cu, net GND
- removed copper zone on F.Cu, net (none)
Other:
- net class Default: trace_width 0.127 -> 0.25; via_dia 0.6 -> 0.8; via_drill 0.3 -> 0.4
- net class Power added: clearance 0.127, trace_width 0.25, via_dia 0.8, via_drill 0.4
- rule trace_min: 0.127 -> 0.25
- board text removed: "MINIMOOD"

Commit message: Use headphone amp IC instead of discrete amp
Parts:
- removed C39: 47u, Capacitor_SMD:CP_Elec_6.3x5.4
- removed J9: Pre_AB_amp, TestPoint:TestPoint_THTPad_D1.0mm_Drill0.5mm
- removed Q1, Q4: BC857B, Package_TO_SOT_SMD:SOT-23
- removed Q2, Q3: BC847B, Package_TO_SOT_SMD:SOT-23
- removed R25, R28, R29, R31: 10k, Resistor_SMD:R_0805_2012Metric
- removed R26: 1k, Resistor_SMD:R_0805_2012Metric
- removed R27: 33, Resistor_SMD:R_0805_2012Metric
- removed R30: 56k, Resistor_SMD:R_0805_2012Metric
- removed R32, R33: 100, Resistor_SMD:R_0805_2012Metric
- removed RV_VOL1: 500k reverse log, Potentiometer_THT:Potentiometer_Alps_RK09K_Single_Horizontal
- added RV1: 10k-dual-reverse-log, Potentiometer_THT:Potentiometer_Alps_RK09L_Double_Horizontal, B.Cu at (178.6, 37.0)
- C21: value 1u -> 2.2u
- C34: value 100n -> 2.2u
- C36: value 47u -> 1u; footprint Capacitor_SMD:CP_Elec_6.3x5.4 -> Capacitor_SMD:C_0805_2012Metric
- C37: value 4.7u -> 100u; footprint Capacitor_SMD:C_0805_2012Metric -> Capacitor_SMD:CP_Elec_6.3x5.4
- C38: value 150p -> 100u; footprint Capacitor_SMD:C_0805_2012Metric -> Capacitor_SMD:CP_Elec_6.3x5.4
- J12: value Post_AB_amp -> Audio_jack_R
- J13: value Audio_out_jack -> Audio_jack_L
- R19: value 1k -> 8.2k
- R22: value 22M -> 8.2k
- R23: value 10k -> 100k
- R24: value 10M -> 100k
- U5: value MCP6002-xSN -> LM4808M_NOPB; footprint Package_SO:SOIC-8_3.9x4.9mm_P1.27mm -> lib:LM4808M&slash_NOPB
- moved J12 39.8 mm to (193.5, 39.6), turned to 270 degrees
- moved R19 31.9 mm to (190.7, 48.0), turned to 180 degrees
- moved R24 26.9 mm to (191.5, 51.0), turned to 270 degrees
- moved C35 24.7 mm to (197.1, 45.4), turned to 0 degrees
- moved C21 24.1 mm to (190.7, 55.1)
- moved R23 23.5 mm to (202.2, 48.9), turned to 270 degrees
- moved C37 22.2 mm to (210.6, 49.5), turned to 0 degrees
- moved C36 22.1 mm to (189.2, 51.0), turned to 90 degrees
- moved C34 20.9 mm to (195.3, 54.1), turned to 180 degrees
- moved U5 19.3 mm to (197.1, 49.5), turned to 0 degrees
- moved C38 17.7 mm to (210.6, 57.4), turned to 0 degrees
- moved R22 16.6 mm to (199.1, 54.1), turned to 0 degrees
- moved J17 3.28 mm to (209.6, 83.3)
- moved C14 2.95 mm to (183.6, 56.1)
- moved J13 0.60 mm to (195.6, 39.6)
Connections:
- C21 pad 1: Net-(C21-Pad1) -> /audio_out/AUDIO_IN
- C36 pad 1: Net-(C36-Pad1) -> GND
- C36 pad 2: GND -> Net-(C36-Pad2)
- C37 pad 1: GND -> Net-(C37-Pad1)
- C37 pad 2: Net-(C37-Pad2) -> /audio_out/Audio_jack_L
- C38 pad 1: /audio_out/audio_post_AB_amp -> Net-(C38-Pad1)
- C38 pad 2: Net-(C38-Pad2) -> /audio_out/Audio_jack_R
- J12 pad 1: /audio_out/audio_post_AB_amp -> /audio_out/Audio_jack_R
- J13 pad 1: /audio_out/Audio_out_jack -> /audio_out/Audio_jack_L
- J6 pad R: /audio_out/Audio_out_jack -> /audio_out/Audio_jack_R
- J6 pad T: /audio_out/Audio_out_jack -> /audio_out/Audio_jack_L
- R18 pad 2: Net-(C21-Pad2) -> /audio_out/AUDIO_IN
- R19 pad 1: Net-(C21-Pad1) -> Net-(R19-Pad1)
- R19 pad 2: /audio_out/AUDIO_IN -> Net-(C21-Pad2)
- R22 pad 1: /audio_out/AUDIO_IN -> Net-(C34-Pad1)
- R22 pad 2: GND -> Net-(R22-Pad2)
- R23 pad 2: Net-(C36-Pad1) -> Net-(C36-Pad2)
- R24 pad 1: Net-(C36-Pad1) -> Net-(C36-Pad2)
- R24 pad 2: Net-(C34-Pad1) -> GND
- U4 pad 7: Net-(C21-Pad2) -> /audio_out/AUDIO_IN
- U5 pad 1: /audio_out/audio_pre_AB_amp -> Net-(C37-Pad1)
- U5 pad 2: Net-(C38-Pad2) -> Net-(R19-Pad1)
- U5 pad 3: Net-(R26-Pad1) -> Net-(C36-Pad2)
- U5 pad 5: GND -> Net-(C36-Pad2)
- U5 pad 6: Net-(U5-Pad6) -> Net-(R22-Pad2)
- U5 pad 7: Net-(U5-Pad6) -> Net-(C38-Pad1)
Routing:
- net Net-(C38-Pad2): track 54.9 -> 0.00 mm
- net /audio_out/audio_post_AB_amp: track 43.8 -> 0.00 mm, vias 2 -> 0
- net Net-(C38-Pad1): track 0.00 -> 41.1 mm
- net /audio_out/audio_pre_AB_amp: track 37.6 -> 0.00 mm, vias 2 -> 0
- net Net-(R27-Pad2): track 35.9 -> 0.00 mm
- net Net-(C37-Pad1): track 0.00 -> 35.7 mm, vias 0 -> 4
- net +5VA: track 211.6 -> 178.5 mm, vias 12 -> 10
- net /audio_out/Audio_jack_R: track 0.00 -> 30.9 mm
- net Net-(R22-Pad2): track 0.00 -> 26.6 mm, vias 0 -> 2
- net /audio_out/Audio_jack_L: track 0.00 -> 23.8 mm
- net /audio_out/Audio_out_jack: track 21.7 -> 0.00 mm
- net GND: track 140.9 -> 119.3 mm, vias 101 -> 106
- net /audio_out/AUDIO_IN: track 27.7 -> 48.4 mm
- net Net-(R19-Pad1): track 0.00 -> 16.7 mm
- net Net-(C36-Pad1): track 14.3 -> 0.00 mm
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Other:
- copper layers 4 -> 2
