File: Hardware/PCB/main_board/MIDI.sch (KiCad schematic (older format))
At the start: 8 parts, among them J2 USB_A, J3 DIN-5_180degree, U3 6N137

Commit message: Add power supply schematics and layout
Parts:
- D1: footprint Diode_THT:D_DO-35_SOD27_P7.62mm_Horizontal -> Diode_SMD:D_SOD-123
- J3: footprint (none) -> lib:MIDI_DIN5
- R8, R9: footprint Resistor_SMD:R_0815_2038Metric -> Resistor_SMD:R_0805_2012Metric
- U3: footprint Package_DIP:DIP-8_W7.62mm -> Package_SO:SOIC-8_3.9x4.9mm_P1.27mm
Changed lines of the file:
@@
 $Descr A4 11693 8268
 encoding utf-8
-Sheet 3 4
+Sheet 2 5
 Title ""
 Date ""
@@
 F 0 "U3" H 5550 2967 50  0000 C CNN
 F 1 "6N137" H 5550 2876 50  0000 C CNN
-F 2 "Package_DIP:DIP-8_W7.62mm" H 5550 2000 50  0001 C CNN
+F 2 "Package_SO:SOIC-8_3.9x4.9mm_P1.27mm" H 5550 2000 50  0001 C CNN
 F 3 "https://docs.broadcom.com/docs/AV02-0940EN" H 4700 3050 50  0001 C CNN
 	1    5550 2500
@@
 F 0 "J3" V 4146 2671 50  0000 R CNN
 F 1 "DIN-5_180degree" V 4055 2671 50  0000 R CNN
-F 2 "" H 4100 2900 50  0001 C CNN
+F 2 "lib:MIDI_DIN5" H 4100 2900 50  0001 C CNN
 F 3 "http://www.mouser.com/ds/2/18/40_c091_abd_e-75918.pdf" H 4100 2900 50  0001 C CNN
 	1    4100 2900
@@
 F 0 "D1" V 4704 2929 50  0000 L CNN
 F 1 "1N4148" V 4795 2929 50  0000 L CNN
-F 2 "Diode_THT:D_DO-35_SOD27_P7.62mm_Horizontal" H 4750 2675 50  0001 C CNN
+F 2 "Diode_SMD:D_SOD-123" H 4750 2675 50  0001 C CNN
 F 3 "https://assets.nexperia.com/documents/data-sheet/1N4148_1N4448.pdf" H 4750 2850 50  0001 C CNN
 	1    4750 2850
@@
 F 0 "R8" V 4243 2500 50  0000 C CNN
 F 1 "220" V 4334 2500 50  0000 C CNN
-F 2 "Resistor_SMD:R_0815_2038Metric" V 4380 2500 50  0001 C CNN
+F 2 "Resistor_SMD:R_0805_2012Metric" V 4380 2500 50  0001 C CNN
 F 3 "~" H 4450 2500 50  0001 C CNN
 	1    4450 2500
@@
 F 0 "R9" V 6443 2500 50  0000 C CNN
 F 1 "10k" V 6534 2500 50  0000 C CNN
-F 2 "Resistor_SMD:R_0815_2038Metric" V 6580 2500 50  0001 C CNN
+F 2 "Resistor_SMD:R_0805_2012Metric" V 6580 2500 50  0001 C CNN
 F 3 "~" H 6650 2500 50  0001 C CNN
 	1    6650 2500

Commit message: Flip connectors, add 3D models
Parts:
- J2: footprint Connector_USB:USB3_A_Molex_48393-001 -> Connector_USB:USB_A_Stewart_SS-52100-001_Horizontal
Changed lines of the file:
@@
 F 0 "J2" H 3407 5317 50  0000 C CNN
 F 1 "USB_A" H 3407 5226 50  0000 C CNN
-F 2 "Connector_USB:USB3_A_Molex_48393-001" H 3500 4800 50  0001 C CNN
+F 2 "Connector_USB:USB_A_Stewart_SS-52100-001_Horizontal" H 3500 4800 50  0001 C CNN
 F 3 " ~" H 3500 4800 50  0001 C CNN
 	1    3350 4850

Commit message: Route PWR
Connections:
- no-connect marks 0 -> 5
Other:
- moved on the sheet: C7
Changed lines of the file:
@@
 L Device:C C7
 U 1 1 5E517904
-P 4950 2100
-F 0 "C7" H 5065 2146 50  0000 L CNN
-F 1 "100n" H 5065 2055 50  0000 L CNN
-F 2 "Capacitor_SMD:C_0805_2012Metric" H 4988 1950 50  0001 C CNN
-F 3 "~" H 4950 2100 50  0001 C CNN
-	1    4950 2100
+P 4950 2050
+F 0 "C7" H 5065 2096 50  0000 L CNN
+F 1 "100n" H 5065 2005 50  0000 L CNN
+F 2 "Capacitor_SMD:C_0805_2012Metric" H 4988 1900 50  0001 C CNN
+F 3 "~" H 4950 2050 50  0001 C CNN
+	1    4950 2050
 	1    0    0    -1
 $EndComp
@@
 L power:+5V #PWR0105
 U 1 1 5E535820
-P 4950 1950
-F 0 "#PWR0105" H 4950 1800 50  0001 C CNN
-F 1 "+5V" H 4965 2123 50  0000 C CNN
-F 2 "" H 4950 1950 50  0001 C CNN
-F 3 "" H 4950 1950 50  0001 C CNN
-	1    4950 1950
+P 4950 1850
+F 0 "#PWR0105" H 4950 1700 50  0001 C CNN
+F 1 "+5V" H 4965 2023 50  0000 C CNN
+F 2 "" H 4950 1850 50  0001 C CNN
+F 3 "" H 4950 1850 50  0001 C CNN
+	1    4950 1850
 	1    0    0    -1
 $EndComp
@@
 Wire Wire Line
 	3650 4950 4050 4950
+Text HLabel 4050 4850 2    50   Output ~ 0
+MIDI_USB_D+
+Text HLabel 4050 4950 2    50   Output ~ 0
+MIDI_USB_D-
+Text Notes 5450 6000 2    118  ~ 24
+USB MIDI
+Wire Notes Line
+	2950 4100 5550 4100
+Wire Notes Line
+	5550 4100 5550 6100
+Wire Notes Line
+	5550 6100 2950 6100
+Wire Notes Line
+	2950 6100 2950 4100
+NoConn ~ 3250 5250
+NoConn ~ 5850 2400
+NoConn ~ 4400 2900
+NoConn ~ 4100 2600
+NoConn ~ 4100 3200
+$Comp
+L power:GND #PWR0110
+U 1 1 5E54748C
+P 3750 5600
+F 0 "#PWR0110" H 3750 5350 50  0001 C CNN
+F 1 "GND" H 3755 5427 50  0000 C CNN
+F 2 "" H 3750 5600 50  0001 C CNN
+F 3 "" H 3750 5600 50  0001 C CNN
+	1    3750 5600
+	1    0    0    -1
+$EndComp
+$Comp
+L power:+5V #PWR0109
+U 1 1 5E547486
+P 3750 5200
+F 0 "#PWR0109" H 3750 5050 50  0001 C CNN
+F 1 "+5V" H 3765 5373 50  0000 C CNN
+F 2 "" H 3750 5200 50  0001 C CNN
+F 3 "" H 3750 5200 50  0001 C CNN
+	1    3750 5200
+	1    0    0    -1
+$EndComp
 $Comp
 L Device:C C6
@@
 	1    0    0    -1
 $EndComp
-$Comp
-L power:+5V #PWR0109
-U 1 1 5E547486
-P 3750 5250
-F 0 "#PWR0109" H 3750 5100 50  0001 C CNN
-F 1 "+5V" H 3765 5423 50  0000 C CNN
-F 2 "" H 3750 5250 50  0001 C CNN
-F 3 "" H 3750 5250 50  0001 C CNN
-	1    3750 5250
-	1    0    0    -1
-$EndComp
-$Comp
-L power:GND #PWR0110
-U 1 1 5E54748C
-P 3750 5550
-F 0 "#PWR0110" H 3750 5300 50  0001 C CNN
-F 1 "GND" H 3755 5377 50  0000 C CNN
-F 2 "" H 3750 5550 50  0001 C CNN
-F 3 "" H 3750 5550 50  0001 C CNN
-	1    3750 5550
-	1    0    0    -1
-$EndComp
-Text HLabel 4050 4850 2    50   Output ~ 0
-MIDI_USB_D+
-Text HLabel 4050 4950 2    50   Output ~ 0
-MIDI_USB_D-
-Text Notes 5450 6000 2    118  ~ 24
-USB MIDI
-Wire Notes Line
-	2950 4100 5550 4100
-Wire Notes Line
-	5550 4100 5550 6100
-Wire Notes Line
-	5550 6100 2950 6100
-Wire Notes Line
-	2950 6100 2950 4100
+Wire Wire Line
+	3750 5550 3750 5600
+Wire Wire Line
+	3750 5250 3750 5200
+Wire Wire Line
+	4950 1850 4950 1900
+Wire Wire Line
+	4950 2200 4950 2250
 $EndSCHEMATC
