File: Hardware/PCB/main_board/power.sch (KiCad schematic (older format))
At the start: 16 parts, among them J21 GND, J22 GND, J23 +5V, J24 +5VA, J4 USB_B, J7 GND, J8 GND, U2 LD1117S33TR_SOT223

Commit message: Re-layout HMI, pre route
Parts:
- removed J23: +5V, Connector_PinHeader_2.54mm:PinHeader_1x01_P2.54mm_Vertical, symbol Connector_Generic:Conn_01x01
- removed J24: +5VA, Connector_PinHeader_2.54mm:PinHeader_1x01_P2.54mm_Vertical, symbol Connector_Generic:Conn_01x01
- added J14: +5V, TestPoint:TestPoint_THTPad_D1.0mm_Drill0.5mm, symbol Connector:TestPoint
- added J23: +3.3V, TestPoint:TestPoint_THTPad_D1.0mm_Drill0.5mm, symbol Connector:TestPoint
- added J24: +5VA, TestPoint:TestPoint_THTPad_D1.0mm_Drill0.5mm, symbol Connector:TestPoint
- J21, J22, J7, J8: footprint Connector_PinHeader_2.54mm:PinHeader_1x01_P2.54mm_Vertical -> TestPoint:TestPoint_THTPad_D1.0mm_Drill0.5mm; symbol Connector_Generic:Conn_01x01 -> Connector:TestPoint
Connections:
- net +3V3: now also J23.1
- net +5V: now also J14.1
- net +5VA: now also J24.1
Other:
- moved on the sheet: C10, C11, C12, C40, C8, C9, FB1, FB2, J4, U2
